File: hardware/KiCad Remote Volume Control.sch (KiCad schematic (older format))
At the start: 25 parts, among them J1 Conn_01x02_Female, J2 AVR-ISP-6, J3 In, J4 Out, U1 ATmega328P-PU, U2 TSOP34S40F, U3 PT2257

Commit message: Make KiCad pathes relative
Parts:
- U3: symbol Project:PT2257 -> KiCad-Remote-Volume-Control-rescue:PT2257-Project
Changed lines of the file:
@@
 	4650 2000 4800 2000
 $Comp
-L Project:PT2257 U3
+L KiCad-Remote-Volume-Control-rescue:PT2257-Project U3
 U 1 1 605F73F9
 P 8950 2300
